File: Hardware/MicroPicoDriveCartridge/MicroPicoDriveCartridge/MicroPicoDriveCartridge.kicad_pcb (KiCad board)
At the start: 2 copper layers, 30.8 x 35 mm, 12 parts, among them J1 Conn_02x08_Odd_Even, SW1 SW_Push, SW2 SW_Push, SW3 SW_Push

Commit message: Updated PCBs
Other:
- board size 30.8 x 35 mm -> 40.3 x 35 mm
Changed lines of the file:
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@@
       (psa4output false)
       (plotreference true)
-      (plotvalue true)
+      (plotvalue false)
       (plotinvisibletext false)
       (sketchpadsonfab false)
@@
       (drillshape 0)
       (scaleselection 1)
-      (outputdirectory "Fabrication/")
+      (outputdirectory "Fabrication_2/")
     )
   )
@@
       (net 21 "unconnected-(SD1-Pad9)") (pinfunction "D2") (pintype "bidirectional+no_connect"))
   )
-  (gr_line (start 127.325 73.375) (end 127.325 108.375) (layer "Edge.Cuts") (width 0.1))
-  (gr_line (start 158.125 108.375) (end 127.325 108.375) (layer "Edge.Cuts") (width 0.1))
-  (gr_line (start 158.125 73.375) (end 158.125 108.375) (layer "Edge.Cuts") (width 0.1))
+  (gr_line (start 127.325 73.375) (end 127.325 100.375) (layer "Edge.Cuts") (width 0.1))
+  (gr_arc (start 162.1 104.35) (mid 162.825185 106.645773) (end 161.15 108.375) (layer "Edge.Cuts") (width 0.1))
+  (gr_line (start 162.1 104.35) (end 158.125 100.375) (layer "Edge.Cuts") (width 0.1))
+  (gr_line (start 161.15 108.375) (end 124.3 108.375) (layer "Edge.Cuts") (width 0.1))
+  (gr_arc (start 124.3 108.375) (mid 122.624834 106.645776) (end 123.35 104.35) (layer "Edge.Cuts") (width 0.1))
+  (gr_line (start 127.325 100.375) (end 123.35 104.35) (layer "Edge.Cuts") (width 0.1))
+  (gr_line (start 158.125 73.375) (end 158.125 100.375) (layer "Edge.Cuts") (width 0.1))
   (segment (start 152.535 88.1) (end 149.575 88.1) (width 0.25) (layer "F.Cu") (net 1))
   (segment (start 136.7908 68.3908) (end 136.7908 86.5653) (width 0.25) (layer "F.Cu") (net 2))
@@
     (polygon
       (pts
-        (xy 160.275 110.8)
-        (xy 123.45 110.8)
-        (xy 123.45 73.4)
-        (xy 160.275 73.4)
+        (xy 170.525 110.8)
+        (xy 114.6 110.8)
+        (xy 114.6 73.4)
+        (xy 170.525 73.4)
       )
     )
